File: pcb/wrx-power-can-hat-FINAL.kicad_sch (KiCad schematic)
At the start: 66 parts, among them J1 ISO_A, J2 Pi_GPIO, J3 OBD-II, J4 CAN_Term, J5 ISP, J6 FAN, J7 Audio, Q1 IRF9540N, Q2 2N7002, Q3 2N7002, U1 LM2596S-5.0, U2 AMS1117-3.3, U3 SN65HVD230, U4 LTV-817S, U5 PCM5142, Y1 8MHz

Commit message: PCB layouts, gerbers, cleanup: Power HAT + CAN HAT ready
PCB Layout Updates:
- Power HAT: Fan control (GPIO12/13), 8 mounting holes, back-layer optimization
- CAN HAT: Complete PCB with GPIO header, MCP2515, OBD-II connector

Gerber Files Added:
- Power HAT gerbers (ready for fabrication)
- CAN HAT gerbers (ready for fabrication)
- DAC/Amp gerbers

Documentation:
- BOM files for all boards
- GPIO wiring documentation
- Footprint assignments

Cleanup:
- Removed 30+ temporary fix scripts
- Removed backup schematic files
- Removed test files

Co-Authored-By: Claude Opus 4.5 <noreply@anthropic.com>
Parts:
- removed C?: 220uF, symbol Device:CP
- removed C? (x2): 100uF, symbol Device:CP
- removed D4: 1N4148, symbol Device:D
- removed U?: ATtiny85, symbol MCU_Microchip_ATtiny:ATtiny85-20PU
- removed U?: MCP2515, symbol Interface_CAN_LIN:MCP2515-I_SO
Connections:
- net +3.3V: now also J1.8 (Pin_8), J2.1 (Pin_1), J2.12 (Pin_12), J2.2 (Pin_2), J2.23 (Pin_23), J2.24 (Pin_24), J2.4 (Pin_4), J2.6 (Pin_6), J2.9 (Pin_9), J3.2 (Pin_2), J3.3 (Pin_3), J3.4 (Pin_4), J3.6 (Pin_6), J5.1 (Pin_1), J5.2 (Pin_2), J6.2 (Pin_2), J7.6 (Pin_6), JP1.2 (Pin_2), Q2.3 (D), Q3.1 (G), R15.2, U1.3 (GND), U3.6 (CANL), U3.8 (Rs), U5.1 (Pin_1), U5.2 (Pin_2), U5.3 (Pin_3), U5.4 (Pin_4), U5.5 (Pin_5), U5.6 (Pin_6); no longer J2.16 (Pin_16), J2.18 (Pin_18), J2.38 (Pin_38), J3.10 (Pin_10), J5.5 (Pin_5)
- net AUDIO_L_OUT: now also R17.2
- net AUDIO_R+: now also C15.1, J7.2 (Pin_2), J7.3 (Pin_3), J7.4 (Pin_4), J7.5 (Pin_5), R16.1, R17.1, R18.1, R19.1
- net AUDIO_R_OUT: now also R18.2, R19.2; no longer C15.1, J7.2 (Pin_2), J7.3 (Pin_3), J7.4 (Pin_4), J7.5 (Pin_5), R16.1, R17.1, R18.1, R19.1
- net FAN_PWM: now also R15.1
- net HEARTBEAT_LED: now also U3.3 (VCC)
- net LED2_ANODE: now also R9.2
- net RESET: now also J3.5 (Pin_5)
- net SPI_MISO: now also J2.21 (Pin_21), J3.1 (Pin_1)
- net TIMER_LED: now also U3.2 (GND)
- net 12V_IGN: now reaches J1.7 (Pin_7)
- net 12V_IGN: now also R6.1, U2.1 (GND)
- net CAN_INT: now reaches J2.22 (Pin_22)
- net +12V: no longer names the net of F1.2, J1.4 (Pin_4), R1.2
- net FAN+: no longer names the net of J6.1 (Pin_1), JP2.2 (Pin_2)
- no-connect marks 0 -> 48
