File: pcb/wrx-power-can-hat-PINTOPIN.kicad_sch (KiCad schematic)
At the start: 66 parts, among them J1 ISO_A, J2 Pi_GPIO, J3 OBD-II, J4 CAN_Term, J5 ISP, J6 FAN, J7 Audio, Q1 IRF9540N, Q2 2N7002, Q3 2N7002, U1 LM2596S-5.0, U2 AMS1117-3.3, U3 SN65HVD230, U4 LTV-817S, U5 PCM5142, Y1 8MHz

Commit message: PCB layouts, gerbers, cleanup: Power HAT + CAN HAT ready
PCB Layout Updates:
- Power HAT: Fan control (GPIO12/13), 8 mounting holes, back-layer optimization
- CAN HAT: Complete PCB with GPIO header, MCP2515, OBD-II connector

Gerber Files Added:
- Power HAT gerbers (ready for fabrication)
- CAN HAT gerbers (ready for fabrication)
- DAC/Amp gerbers

Documentation:
- BOM files for all boards
- GPIO wiring documentation
- Footprint assignments

Cleanup:
- Removed 30+ temporary fix scripts
- Removed backup schematic files
- Removed test files

Co-Authored-By: Claude Opus 4.5 <noreply@anthropic.com>
Parts:
- removed C?: 220uF, symbol Device:CP
- removed C? (x2): 100uF, symbol Device:CP
- removed D4: 1N4148, symbol Device:D
- removed U?: ATtiny85, symbol MCU_Microchip_ATtiny:ATtiny85-20PU
- removed U?: MCP2515, symbol Interface_CAN_LIN:MCP2515-I_SO
Connections:
- net at C1.1, C10.1, C10.2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: now also D2.2 (A), D3.1 (K), D3.2 (A), LED2.1 (K), R13.1, Y1.2; no longer C1.2, D1.1 (A1), F1.1, LED3.2 (A), R14.1, R2.2, Y1.1
- net at D2.1 (K): now also C1.2, D1.2 (A2), F1.1, R2.2
- net at LED2.2 (A): now also LED3.2 (A), R14.1
- no-connect marks 0 -> 7
