File: pcb/boards/power-hat/power-hat.kicad_sch (KiCad schematic)
At the start: 40 parts, among them J1 ISO_A, J2 Raspberry_Pi_GPIO, J3 ISP, J4 FAN, Q1 IRLB8721PBF, Q2 2N7002, Q3 2N7002, U1 TPS54560BDDA, U2 LTV-817S, U3 attiny85, Y1 16Mhz Crystal

Commit message: Wire ATtiny85 status signals to Pi GPIO header
- Connect U3 PB0 (HEARTBEAT_LED) to J2 Pin 11 (GPIO17)
- Connect U3 PB1 (TIMER_LED) to J2 Pin 13 (GPIO27)
- Add GPIO_ALLOCATION.md documenting pin usage across all 3 HAT boards
- Update README.md with GPIO references and new fix scripts (v12-v14)

This allows the Pi to monitor ATtiny85 power management status signals
through the stackable header interface.

Co-Authored-By: Claude Opus 4.5 <noreply@anthropic.com>
Connections:
- net 12V_IGN is gone; now on net 12V_FUSED: C9.1, D2.2 (A), U1.2 (VIN), U1.3 (EN)
- net GROUND is gone; now on net 12V_ACC: J1.8 (Pin_8)
- net +3.3V: now also R8.1
- net 12V_ACC: now also J1.2 (Pin_2); no longer J1.7 (Pin_7)
- net 12V_FUSED: now also F1.2, J1.1 (Pin_1), J1.3 (Pin_3), J1.4 (Pin_4), R6.1
- net 12V_SWITCHED: now also Q1.3 (S)
- net FAN_PWM: now also R10.1
- net GATE_CTRL: now also R5.2, R8.2
- net GND: now also C_COMP1.2, J1.5 (Pin_5), J1.6 (Pin_6), J1.7 (Pin_7), R10.2, R6.2, R_RT1.2
- net XTAL1: now also Y1.1
- net XTAL2: now also Y1.2
- net FAN+: now reaches J4.1 (Pin_1)
- no-connect marks 27 -> 38
