File: pcb/boards/dac-amp/dac_amp.kicad_sch (KiCad schematic)
At the start: 43 parts, among them J1 I2S_Input, J2 12V_Input, J3 Conn_01x04, J4 Conn_01x04, J7 40-Pin_GPIO, U1 PCM5142, U2 AMS1117-3.3, U3 TPA3116D2DAD, U4 TPA3116D2DAD

Commit message: DAC/Amp HAT PCB: Ready for PCBA manufacturing
- PCB fully routed via FreeRouting auto-router
- DRC clean: 0 unconnected pads, 0 errors (warnings are cosmetic)
- Power traces widened: +12V @ 1.0mm, speaker outputs @ 0.75mm
- Thermal vias added under U3 and U4 (6-8 vias each)
- Fiducials added for pick-and-place assembly
- GND copper pour on back layer for thermal dissipation
- BOM with manufacturer part numbers (dac_amp_bom.csv)
- Gerbers and placement files generated for PCBWay

Manufacturing notes:
- Recommend 2oz copper for power handling
- ENIG surface finish for PCBA
- Double-sided assembly (components on front and back)

Co-Authored-By: Claude Opus 4.5 <noreply@anthropic.com>
Parts:
- J3, J4: footprint (none) -> TerminalBlock_Phoenix:TerminalBlock_Phoenix_PT-1,5-4-3.5-H_1x04_P3.50mm_Horizontal
- U3, U4: footprint Package_SO:HTSSOP-32-1EP_6.1x11mm_P0.65mm_EP5.2x5.2mm -> Package_SO:Texas_DAD0032A_HTSSOP-32_6.1x11mm_P0.65mm_TopEP3.71x3.81mm
Changed lines of the file:
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@@
 			)
 		)
-		(property "Footprint" "Package_SO:HTSSOP-32-1EP_6.1x11mm_P0.65mm_EP5.2x5.2mm"
+		(property "Footprint" "Package_SO:Texas_DAD0032A_HTSSOP-32_6.1x11mm_P0.65mm_TopEP3.71x3.81mm"
 			(at 182.88 110.49 0)
 			(effects
@@
 			)
 		)
-		(property "Footprint" ""
+		(property "Footprint" "TerminalBlock_Phoenix:TerminalBlock_Phoenix_PT-1,5-4-3.5-H_1x04_P3.50mm_Horizontal"
 			(at 234.95 179.07 0)
 			(effects
@@
 			)
 		)
-		(property "Footprint" "Package_SO:HTSSOP-32-1EP_6.1x11mm_P0.65mm_EP5.2x5.2mm"
+		(property "Footprint" "Package_SO:Texas_DAD0032A_HTSSOP-32_6.1x11mm_P0.65mm_TopEP3.71x3.81mm"
 			(at 182.88 215.9 0)
 			(effects
@@
 			)
 		)
-		(property "Footprint" ""
+		(property "Footprint" "TerminalBlock_Phoenix:TerminalBlock_Phoenix_PT-1,5-4-3.5-H_1x04_P3.50mm_Horizontal"
 			(at 234.95 158.75 0)
 			(effects
